File: ESC_PLC.kicad_pcb (KiCad board)
At the start: 2 copper layers, 145 parts, among them J1 RJ45_Amphenol_RJMG1BD3B8K1ANR, J2 RJ45_Amphenol_RJMG1BD3B8K1ANR, J3 Screw_Terminal_01x05, J4 Screw_Terminal_01x03, U1 stm32G4, U3 MIC4604YM, U4 MIC4604YM, U5 MIC4604YM, Y1 LFXTAL085880

Commit message: pcb gesorteerd
al de main blokken bij elkaar gezet
Parts:
- added C82: 8p, Capacitor_SMD:C_0603_1608Metric, F.Cu at (336.8, 108.8)
- added C83: 8p, Capacitor_SMD:C_0603_1608Metric, F.Cu at (336.8, 111.3)
- added Y2: 8Mhz, Footprintsymbolen_samen:25Mhz crystal 8pF, F.Cu at (331.1, 109.6)
- Y1: value LFXTAL085880 -> 25Mhz
- moved Y1 261.6 mm to (124.7, 144.1)
- moved C45 226.2 mm to (147.9, 155.0)
- moved C46 226.2 mm to (147.9, 157.5)
- moved J2 226.2 mm to (159.7, 135.5)
- moved R1 226.2 mm to (147.9, 170.1)
- moved R10 226.2 mm to (151.9, 167.6)
- moved R2 226.2 mm to (147.9, 172.6)
- moved R3 226.2 mm to (147.9, 175.1)
- moved R4 226.2 mm to (147.9, 177.6)
- moved R5 226.2 mm to (151.9, 155.0)
- moved R6 226.2 mm to (151.9, 157.5)
- moved R7 226.2 mm to (151.9, 160.1)
- moved R8 226.2 mm to (151.9, 162.6)
- moved R9 226.2 mm to (151.9, 165.1)
- moved U2 226.2 mm to (161.7, 161.2)
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Connections:
- U1 pad 5: unconnected-(U1-PE6-Pad5) -> /µcontroller/OSC_IN
- U1 pad 6: unconnected-(U1-PF1-Pad6) -> /µcontroller/OSC_OUT
Routing:
- net GND: track 0.00 -> 32.5 mm, vias 0 -> 7
- net +3V3: track 0.00 -> 13.2 mm
- net unconnected-(U1-PB10-Pad30): track 0.00 -> 8.47 mm
- net Net-(U1-VREF+): track 0.00 -> 6.77 mm
Other:
- board outline added: 80 x 72 mm

Commit message: al de main blokken bij elkaar gezet op juiste plaats
Parts:
- removed C41: 100n, Capacitor_SMD:C_0603_1608Metric
- removed C42: 1µ, Capacitor_SMD:C_0603_1608Metric
- added D5: NUP2105L, Package_TO_SOT_SMD:SOT-23, F.Cu at (388.8, 100.6)
- C66, C67: footprint Capacitor_SMD:C_0603_1608Metric -> Capacitor_SMD:CP_Elec_10x10
- moved C58 126.7 mm to (384.7, 100.6)
- moved R23 126.1 mm to (382.3, 98.8), turned to -90 degrees
- moved R24 125.7 mm to (382.3, 102.5), turned to -90 degrees
- moved C57 113.6 mm to (371.6, 100.6), turned to 90 degrees
- moved U6 111.5 mm to (374.3, 98.8)
- moved C56 111.2 mm to (370.1, 100.7), turned to 90 degrees
- moved C61 57.0 mm to (215.4, 134.4), turned to -90 degrees
- moved FB1 51.4 mm to (98.6, 174.8), turned to 90 degrees
- moved FB3 50.3 mm to (98.3, 156.7), turned to -90 degrees
- moved FB2 49.4 mm to (98.6, 166.7), turned to 90 degrees
- moved U2 49.0 mm to (112.8, 164.4), turned to 90 degrees
- moved R1 47.6 mm to (100.7, 164.1), turned to 180 degrees
- moved C62 44.4 mm to (221.1, 127.4)
- moved U7 44.0 mm to (234.1, 125.9)
- moved C63 43.5 mm to (221.1, 128.9)
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Connections:
- C82 pad 1: /µcontroller/OSC_IN -> /µcontroller/OSC_OUT
- Y1 pad 4: unconnected-(Y1-GND-Pad4) -> GND
- Y2 pad 3: /µcontroller/OSC_IN -> /µcontroller/OSC_OUT
- Y2 pad 4: unconnected-(Y2-GND-Pad4) -> GND
Routing:
- net GND: track 32.5 -> 117.3 mm, vias 7 -> 14
- net +3V3: track 13.2 -> 65.3 mm
- net /µcontroller/OSC_IN: track 0.00 -> 18.8 mm
- net /Ethercat Sheet/VDDCR: track 0.00 -> 18.5 mm
- net /Ethercat Sheet/VDD1212TX: track 0.00 -> 16.5 mm
- net /µcontroller/OSC_OUT: track 0.00 -> 14.2 mm
- net /Ethercat Sheet/OSCO: track 0.00 -> 13.1 mm
- net /Ethercat Sheet/TXRX2: track 0.00 -> 12.7 mm
- net /Ethercat Sheet/RXPB: track 0.00 -> 11.9 mm
- net /Ethercat Sheet/RXNB: track 0.00 -> 11.7 mm
- net /Ethercat Sheet/TXPB: track 0.00 -> 11.6 mm
- net /Ethercat Sheet/TXNB: track 0.00 -> 11.6 mm
- net /Ethercat Sheet/OSCI: track 0.00 -> 11.0 mm
- net /Ethercat Sheet/TXRX1: track 0.00 -> 10.3 mm
- net /CAN/CANL: track 0.00 -> 10.3 mm
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
Commit message: connector
connector toegevoegd en wat pinnen aangepast
Parts:
- D4: value 1N5819 -> SS210; footprint Diode_THT:D_DO-41_SOD81_P10.16mm_Horizontal -> Diode_SMD:D_SMA
- IC1: value ~ -> 24AA32AF
- IC2, IC3: value ~ -> MagI3C Power Module 171013201
- Q1, Q2, Q3, Q4, Q5, Q6: value ~ -> STB100N10F7
- U1: value stm32G4 -> stm32G474
- U6: value ~ -> TCAN334GD
- U7: value ~ -> TL2575HV-12
- moved D4 2.10 mm to (208.5, 116.6)
Connections:
- U2 pad 52: /Ethercat Sheet/RXPA -> /Ethercat Sheet/TXNA
- U2 pad 53: /Ethercat Sheet/RXNA -> /Ethercat Sheet/TXPA
- U2 pad 54: /Ethercat Sheet/TXPA -> /Ethercat Sheet/RXNA
- U2 pad 55: /Ethercat Sheet/TXNA -> /Ethercat Sheet/RXPA
