File: Ethercat.kicad_sch (KiCad schematic)
At the start: 51 parts, among them J1 RJ45_Amphenol_RJMG1BD3B8K1ANR, J2 RJ45_Amphenol_RJMG1BD3B8K1ANR, Y1 25Mhz

Commit message: al de main blokken bij elkaar gezet op juiste plaats
Parts:
- removed C41: 100n, Capacitor_SMD:C_0603_1608Metric, symbol Device:C
- removed C42: 1µ, Capacitor_SMD:C_0603_1608Metric, symbol Device:C
Connections:
- net GND: now also Y1.4 (GND); no longer Y1.2 (GND)
Other:
- moved on the sheet: C39, C40

Commit message: connector
connector toegevoegd en wat pinnen aangepast
Parts:
- IC1: value (none) -> 24AA32AF
Connections:
- net GND: now also Y1.2 (GND)
- net RXNA: now also U2.54 (RXNA); no longer U2.53 (TXPA)
- net RXPA: now also U2.55 (RXPA); no longer U2.52 (TXNA)
- net TXNA: now also U2.52 (TXNA); no longer U2.55 (RXPA)
- net TXPA: now also U2.53 (TXPA); no longer U2.54 (RXNA)
Other:
- moved on the sheet: C43, C44, U2, Y1
Changed lines of the file:
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@@
 	)
 	(rectangle
-		(start 255.27 176.657)
-		(end 294.64 208.153)
+		(start 254.635 176.657)
+		(end 294.005 208.153)
 		(stroke
 			(width 0)
@@
 	(text "Crystal\n"
 		(exclude_from_sim no)
-		(at 262.636 179.324 0)
+		(at 262.001 179.324 0)
 		(effects
 			(font
@@
 	)
 	(junction
-		(at 265.43 186.69)
+		(at 264.795 186.69)
 		(diameter 0)
 		(color 0 0 0 0)
@@
 	)
 	(junction
-		(at 281.94 186.69)
+		(at 281.305 186.69)
 		(diameter 0)
 		(color 0 0 0 0)
@@
 	)
 	(junction
+		(at 273.685 191.77)
+		(diameter 0)
+		(color 0 0 0 0)
+	)
+	(junction
 		(at 89.535 162.56)
 		(diameter 0)
@@
 	)
 	(junction
-		(at 274.32 191.73)
+		(at 273.685 191.73)
 		(diameter 0)
 		(color 0 0 0 0)
@@
 	(wire
 		(pts
-			(xy 278.13 186.69) (xy 281.94 186.69)
+			(xy 277.495 186.69) (xy 281.305 186.69)
 		)
 		(stroke
@@
 	(wire
 		(pts
+			(xy 273.685 191.77) (xy 273.685 198.12)
+		)
+		(stroke
+			(width 0)
+			(type default)
+		)
+	)
+	(wire
+		(pts
 			(xy 156.21 104.775) (xy 156.21 107.95)
 		)
@@
 	(wire
 		(pts
-			(xy 281.94 186.69) (xy 290.83 186.69)
+			(xy 281.305 186.69) (xy 290.195 186.69)
 		)
 		(stroke
@@
 	(wire
 		(pts
-			(xy 281.94 196.215) (xy 281.94 198.12)
+			(xy 281.305 196.215) (xy 281.305 198.12)
 		)
 		(stroke
@@
 	(wire
 		(pts
-			(xy 260.35 186.69) (xy 265.43 186.69)
+			(xy 259.715 186.69) (xy 264.795 186.69)
 		)
 		(stroke
@@
 	(wire
 		(pts
-			(xy 270.51 186.69) (xy 265.43 186.69)
+			(xy 269.875 186.69) (xy 264.795 186.69)
 		)
 		(stroke
@@
 	(wire
 		(pts
-			(xy 281.94 186.69) (xy 281.94 188.595)
+			(xy 281.305 186.69) (xy 281.305 188.595)
 		)
 		(stroke
@@
 	(wire
 		(pts
-			(xy 274.32 190.5) (xy 274.32 198.12)
+			(xy 273.685 190.5) (xy 273.685 191.77)
 		)
 		(stroke
@@
 	(wire
 		(pts
-			(xy 265.43 196.215) (xy 265.43 198.12)
+			(xy 264.795 196.215) (xy 264.795 198.12)
 		)
 		(stroke
@@
 	(wire
 		(pts
-			(xy 265.43 186.69) (xy 265.43 188.595)
+			(xy 264.795 186.69) (xy 264.795 188.595)
 		)
 		(stroke
@@
 		)
 	)
-	(label "TXNA"
+	(label "RXPA"
 		(at 93.345 138.43 0)
 		(effects
@@
 		)
 	)
-	(label "RXNA"
+	(label "TXPA"
 		(at 93.345 133.35 0)
 		(effects
@@
 	)
 	(label "OSCI"
-		(at 260.35 186.69 0)
+		(at 259.715 186.69 0)
 		(effects
 			(font
@@
 		)
 	)
-	(label "TXPA"
+	(label "RXNA"
 		(at 93.345 135.89 0)
 		(effects
@@
 		)
 	)
-	(label "RXPA"
+	(label "TXNA"
 		(at 93.345 130.81 0)
 		(effects
@@
 	)
 	(label "OSCO"
-		(at 285.75 186.69 0)
+		(at 285.115 186.69 0)
 		(effects
 			(font
@@
 	(symbol
 		(lib_id "Device:C")
-		(at 265.43 192.405 0)
+		(at 264.795 192.405 0)
 		(unit 1)
 		(body_style 1)
@@
 		(dnp no)
 		(property "Reference" "C43"
-			(at 266.7 190.119 0)
+			(at 266.065 190.119 0)
 			(show_name no)
 			(do_not_autoplace no)
@@
 		)
 		(property "Value" "8p"
-			(at 266.446 194.691 0)
+			(at 265.811 194.691 0)
 			(show_name no)
 			(do_not_autoplace no)
@@
 		)
 		(property "Footprint" "Capacitor_SMD:C_0603_1608Metric"
-			(at 266.3952 196.215 0)
+			(at 265.7602 196.215 0)
 			(hide yes)
 			(show_name no)
@@
 		)
 		(property "Datasheet" ""
-			(at 265.43 192.405 0)
+			(at 264.795 192.405 0)
 			(hide yes)
 			(show_name no)
@@
 		)
 		(property "Description" "Unpolarized capacitor"
-			(at 265.43 192.405 0)
+			(at 264.795 192.405 0)
 			(hide yes)
 			(show_name no)
@@
 		(dnp no)
 		(property "Reference" "U2"
-			(at 106.68 108.966 0)
+			(at 106.426 106.172 0)
 			(show_name no)
 			(do_not_autoplace no)
@@
 	(symbol
 		(lib_id "Schemasymbolen_samen:25Mhz_crystal")
-		(at 270.51 185.42 0)
+		(at 269.875 185.42 0)
 		(unit 1)
 		(body_style 1)
@@
 		(dnp no)
 		(property "Reference" "Y1"
-			(at 273.05 182.626 0)
+			(at 272.415 182.626 0)
 			(show_name no)
 			(do_not_autoplace no)
@@
 		)
 		(property "Value" "25Mhz"
-			(at 278.511 182.626 0)
+			(at 277.876 182.626 0)
 			(show_name no)
 			(do_not_autoplace no)
@@
 		)
 		(property "Footprint" "Footprintsymbolen_samen:25Mhz crystal 8pF"
-			(at 265.938 175.006 0)
+			(at 265.303 175.006 0)
 			(hide yes)
 			(show_name no)
@@
 		)
 		(property "Datasheet" "https://www.mouser.be/datasheet/3/1460/1/LFXTAL085880.pdf"
-			(at 286.512 179.832 0)
+			(at 285.877 179.832 0)
 			(hide yes)
 			(show_name no)
@@
 		)
 		(property "Description" "LFXTAL085880"
-			(at 270.51 185.42 0)
+			(at 269.875 185.42 0)
 			(hide yes)
 			(show_name no)
@@
 	(symbol
 		(lib_id "Device:C")
-		(at 281.94 192.405 0)
+		(at 281.305 192.405 0)
 		(unit 1)
 		(body_style 1)
@@
 		(dnp no)
 		(property "Reference" "C44"
-			(at 283.21 190.119 0)
+			(at 282.575 190.119 0)
 			(show_name no)
 			(do_not_autoplace no)
@@
 		)
 		(property "Value" "8p"
-			(at 282.956 194.691 0)
+			(at 282.321 194.691 0)
 			(show_name no)
 			(do_not_autoplace no)
@@
 		)
 		(property "Footprint" "Capacitor_SMD:C_0603_1608Metric"
-			(at 282.9052 196.215 0)
+			(at 282.2702 196.215 0)
 			(hide yes)
 			(show_name no)
@@
 		)
 		(property "Datasheet" ""
-			(at 281.94 192.405 0)
+			(at 281.305 192.405 0)
 			(hide yes)
 			(show_name no)
@@
 		)
 		(property "Description" "Unpolarized capacitor"
-			(at 281.94 192.405 0)
+			(at 281.305 192.405 0)
 			(hide yes)
 			(show_name no)
@@
 	(symbol
 		(lib_id "power:GNDREF")
-		(at 274.32 198.12 0)
+		(at 273.685 198.12 0)
 		(unit 1)
 		(body_style 1)
@@
 		(dnp no)
 		(property "Reference" "#PWR041"
-			(at 274.32 204.47 0)
+			(at 273.685 204.47 0)
 			(hide yes)
 			(show_name no)
@@
 		)
 		(property "Value" "GND"
-			(at 274.32 201.93 0)
+			(at 273.685 201.93 0)
 			(show_name no)
 			(do_not_autoplace no)
@@
 		)
 		(property "Footprint" ""
-			(at 274.32 198.12 0)
+			(at 273.685 198.12 0)
 			(hide yes)
 			(show_name no)
@@
 		)
 		(property "Datasheet" ""
-			(at 274.32 198.12 0)
+			(at 273.685 198.12 0)
 			(hide yes)
 			(show_name no)
@@
 		)
 		(property "Description" "Power symbol creates a global label with name \"GNDREF\" , reference supply ground"
-			(at 274.32 198.12 0)
+			(at 273.685 198.12 0)
 			(hide yes)
 			(show_name no)
@@
 		(dnp no)
 		(property "Reference" "IC1"
-			(at 275.59 144.145 0)
+			(at 275.59 141.732 0)
 			(show_name no)
 			(do_not_autoplace no)
@@
 			)
 		)
-		(property "Value" ""
-			(at 273.05 144.145 0)
+		(property "Value" "24AA32AF"
+			(at 278.765 144.145 0)
 			(show_name no)
 			(do_not_autoplace no)
@@
 	(symbol
 		(lib_id "power:GNDREF")
-		(at 265.43 198.12 0)
+		(at 264.795 198.12 0)
 		(unit 1)
 		(body_style 1)
@@
 		(dnp no)
 		(property "Reference" "#PWR039"
-			(at 265.43 204.47 0)
+			(at 264.795 204.47 0)
 			(hide yes)
 			(show_name no)
@@
 		)
 		(property "Value" "GND"
-			(at 265.43 201.93 0)
+			(at 264.795 201.93 0)
 			(show_name no)
 			(do_not_autoplace no)
@@
 		)
 		(property "Footprint" ""
-			(at 265.43 198.12 0)
+			(at 264.795 198.12 0)
 			(hide yes)
 			(show_name no)
@@
 		)
 		(property "Datasheet" ""
-			(at 265.43 198.12 0)
+			(at 264.795 198.12 0)
 			(hide yes)
 			(show_name no)
@@
 		)
 		(property "Description" "Power symbol creates a global label with name \"GNDREF\" , reference supply ground"
-			(at 265.43 198.12 0)
+			(at 264.795 198.12 0)
 			(hide yes)
 			(show_name no)
@@
 	(symbol
 		(lib_id "power:GNDREF")
-		(at 281.94 198.12 0)
+		(at 281.305 198.12 0)
 		(unit 1)
 		(body_style 1)
@@
 		(dnp no)
 		(property "Reference" "#PWR042"
-			(at 281.94 204.47 0)
+			(at 281.305 204.47 0)
 			(hide yes)
 			(show_name no)
@@
 		)
 		(property "Value" "GND"
-			(at 281.94 201.93 0)
+			(at 281.305 201.93 0)
 			(show_name no)
 			(do_not_autoplace no)
@@
 		)
 		(property "Footprint" ""
-			(at 281.94 198.12 0)
+			(at 281.305 198.12 0)
 			(hide yes)
 			(show_name no)
@@
 		)
 		(property "Datasheet" ""
-			(at 281.94 198.12 0)
+			(at 281.305 198.12 0)
 			(hide yes)
 			(show_name no)
@@
 		)
 		(property "Description" "Power symbol creates a global label with name \"GNDREF\" , reference supply ground"
-			(at 281.94 198.12 0)
+			(at 281.305 198.12 0)
 			(hide yes)
 			(show_name no)

Commit message: schema's finalized
Parts:
- added R34: 10k, Resistor_SMD:R_0603_1608Metric, symbol Device:R
Connections:
- net +3V3: now also R34.2
- net RST#: no longer names the net of U2.11 (RST#)
- net RST#: now also R34.1
Other:
- moved on the sheet: C30
Changed lines of the file:
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@@
 	(text_box "1µ moet 0.1ohm ESR\n"
 		(exclude_from_sim no)
-		(at 139.573 190.206 0)
+		(at 138.43 192.492 0)
 		(size 9.144 4.358)
 		(margins 0.9525 0.9525 0.9525 0.9525)
@@
 	(wire
 		(pts
+			(xy 148.59 172.72) (xy 148.59 181.61)
+		)
+		(stroke
+			(width 0)
+			(type default)
+		)
+	)
+	(wire
+		(pts
 			(xy 52.07 151.13) (xy 52.07 152.4)
 		)
@@
 	(wire
 		(pts
-			(xy 142.24 180.34) (xy 142.24 179.07)
+			(xy 141.605 180.34) (xy 141.605 179.07)
+		)
+		(stroke
+			(width 0)
+			(type default)
+		)
+	)
+	(wire
+		(pts
+			(xy 156.21 196.85) (xy 156.21 196.215)
 		)
 		(stroke
@@
 	(wire
 		(pts
+			(xy 148.59 196.85) (xy 156.21 196.85)
+		)
+		(stroke
+			(width 0)
+			(type default)
+		)
+	)
+	(wire
+		(pts
 			(xy 89.535 163.83) (xy 89.535 162.56)
 		)
@@
 	(wire
 		(pts
-			(xy 135.89 187.96) (xy 142.24 187.96)
+			(xy 135.89 187.96) (xy 141.605 187.96)
 		)
 		(stroke
@@
 	(wire
 		(pts
+			(xy 148.59 189.23) (xy 148.59 196.85)
+		)
+		(stroke
+			(width 0)
+			(type default)
+		)
+	)
+	(wire
+		(pts
 			(xy 303.53 151.765) (xy 303.53 142.875)
 		)
@@
 	(wire
 		(pts
-			(xy 135.89 179.07) (xy 142.24 179.07)
+			(xy 135.89 179.07) (xy 141.605 179.07)
 		)
 		(stroke
@@
 	(wire
 		(pts
-			(xy 148.59 172.72) (xy 148.59 175.26)
-		)
-		(stroke
-			(width 0)
-			(type default)
-		)
-	)
-	(wire
-		(pts
 			(xy 121.285 192.405) (xy 121.285 190.5)
 		)
@@
 		)
 	)
-	(hierarchical_label "RST#"
-		(shape input)
-		(at 148.59 175.26 270)
-		(effects
-			(font
-				(size 1.27 1.27)
-			)
-			(justify right)
-		)
-	)
 	(hierarchical_label "IRQ"
 		(shape output)
@@
 	)
 	(symbol
+		(lib_id "power:+3V3")
+		(at 156.21 196.215 0)
+		(unit 1)
+		(body_style 1)
+		(exclude_from_sim no)
+		(in_bom yes)
+		(on_board yes)
+		(in_pos_files yes)
+		(dnp no)
+		(property "Reference" "#PWR0119"
+			(at 156.21 200.025 0)
+			(hide yes)
+			(show_name no)
+			(do_not_autoplace no)
+			(effects
+				(font
+					(size 1.27 1.27)
+				)
+			)
+		)
+		(property "Value" "+3V3"
+			(at 156.21 192.151 0)
+			(show_name no)
+			(do_not_autoplace no)
+			(effects
+				(font
+					(size 1.27 1.27)
+				)
+			)
+		)
+		(property "Footprint" "Package_DIP:DIP-24_W7.62mm"
+			(at 156.21 196.215 0)
+			(hide yes)
+			(show_name no)
+			(do_not_autoplace no)
+			(effects
+				(font
+					(size 1.27 1.27)
+				)
+			)
+		)
+		(property "Datasheet" ""
+			(at 156.21 196.215 0)
+			(hide yes)
+			(show_name no)
+			(do_not_autoplace no)
+			(effects
+				(font
+					(size 1.27 1.27)
+				)
+			)
+		)
+		(property "Description" "Power symbol creates a global label with name \"+3V3\""
+			(at 156.21 196.215 0)
+			(hide yes)
+			(show_name no)
+			(do_not_autoplace no)
+			(effects
+				(font
+					(size 1.27 1.27)
+				)
+			)
+		)
+		(pin "1"
+		)
+		(instances
+			(project "ESC_PLC"
+				(path "/5bd3bb6f-fe53-443c-806c-077e2bbb5d14/f038ea58-2b1a-4d87-b3c8-8d32ce4ec05b"
+					(reference "#PWR0119")
+					(unit 1)
+				)
+			)
+		)
+	)
+	(symbol
 		(lib_id "EEPROM:579-24LC32AFT-I/SN")
 		(at 273.05 144.145 0)
@@
 	)
 	(symbol
+		(lib_id "Device:R")
+		(at 148.59 185.42 0)
+		(unit 1)
+		(body_style 1)
+		(exclude_from_sim no)
+		(in_bom yes)
+		(on_board yes)
+		(in_pos_files yes)
+		(dnp no)
+		(property "Reference" "R34"
+			(at 148.717 189.23 0)
+			(show_name no)
+			(do_not_autoplace no)
+			(effects
+				(font
+					(size 1.27 1.27)
+				)
+				(justify left)
+			)
+		)
+		(property "Value" "10k"
+			(at 149.098 191.135 0)
+			(show_name no)
+			(do_not_autoplace no)
+			(effects
+				(font
+					(size 1.27 1.27)
+				)
+				(justify left)
+			)
+		)
+		(property "Footprint" "Resistor_SMD:R_0603_1608Metric"
+			(at 146.812 185.42 90)
+			(hide yes)
+			(show_name no)
+			(do_not_autoplace no)
+			(effects
+				(font
+					(size 1.27 1.27)
+				)
+			)
+		)
+		(property "Datasheet" ""
+			(at 148.59 185.42 0)
+			(hide yes)
+			(show_name no)
+			(do_not_autoplace no)
+			(effects
+				(font
+					(size 1.27 1.27)
+				)
+			)
+		)
+		(property "Description" "Resistor"
+			(at 148.59 185.42 0)
+			(hide yes)
+			(show_name no)
+			(do_not_autoplace no)
+			(effects
+				(font
+					(size 1.27 1.27)
+				)
+			)
+		)
+		(pin "2"
+		)
+		(pin "1"
+		)
+		(instances
+			(project "ESC_PLC"
+				(path "/5bd3bb6f-fe53-443c-806c-077e2bbb5d14/f038ea58-2b1a-4d87-b3c8-8d32ce4ec05b"
+					(reference "R34")
+					(unit 1)
+				)
+			)
+		)
+	)
+	(symbol
 		(lib_id "power:+3V3")
 		(at 114.935 179.07 0)
@@
 	(symbol
 		(lib_id "Device:C")
-		(at 142.24 184.15 0)
+		(at 141.605 184.15 0)
 		(unit 1)
 		(body_style 1)
@@
 		(dnp no)
 		(property "Reference" "C30"
-			(at 142.748 182.118 0)
+			(at 142.113 182.118 0)
 			(show_name no)
 			(do_not_autoplace no)
@@
 		)
 		(property "Value" "1µ"
-			(at 142.748 186.436 0)
+			(at 142.113 186.436 0)
 			(show_name no)
 			(do_not_autoplace no)
@@
 		)
 		(property "Footprint" "Capacitor_SMD:C_0603_1608Metric"
-			(at 143.2052 187.96 0)
+			(at 142.5702 187.96 0)
 			(hide yes)
 			(show_name no)
@@
 		)
 		(property "Datasheet" ""
-			(at 142.24 184.15 0)
+			(at 141.605 184.15 0)
 			(hide yes)
 			(show_name no)
@@
 		)
 		(property "Description" "Unpolarized capacitor"
-			(at 142.24 184.15 0)
+			(at 141.605 184.15 0)
 			(hide yes)
 			(show_name no)
